Commit message: Update for compatability with dyno_hsr

File: robots/hsrb4s.urdf (robot description, URDF)
Before this commit: robot hsrb, 45 links, 44 joints
Links:
- removed link head_rgbd_sensor_gazebo_frame
- added link head_rgbd_sensor_frame
Joints:
- removed joint head_rgbd_sensor_gazebo_frame_joint
- added joint head_rgbd_sensor_frame_joint: type fixed, parent head_rgbd_sensor_link, child head_rgbd_sensor_frame, origin xyz=0 0 0 rpy=0.0 0.0 0.0

File: robots/hsrb4s.urdf.xacro (robot description, xacro)
@@ -60,6 +60,21 @@
     </xacro:hsrb_hand>
     <gazebo>
+      <!--
+      <plugin name="object_controller" filename="libgazebo_ros_planar_move.so">
+          <commandTopic>cmd_vel</commandTopic>
+          <odometryTopic>/odom</odometryTopic>
+          <odometryFrame>odom</odometryFrame>
+          <odometryRate>20.0</odometryRate>
+          <robotBaseFrame>base_footprint</robotBaseFrame>
+        </plugin>
+ -->
+        <!--
         <plugin name="${robot_name}_ros_control" filename="lib${robot_name}_gazebo_ros_control.so">
             <robotNamespace>${robot_name}</robotNamespace>
+        </plugin>
+        -->
+        <plugin name="gazebo_ros_control" filename="libgazebo_ros_control.so">
+            <robotNamespace>${robot_name}</robotNamespace>
+            <robotSimType>gazebo_ros_control/DefaultRobotHWSim</robotSimType>
         </plugin>
         <plugin name="${robot_name}_p3d_ground_truth" filename="libgazebo_ros_p3d.so">

File: urdf/base_v2/base.gazebo.xacro (robot description, xacro)
@@ -35,4 +35,9 @@
         <gazebo_link name="${prefix}_range_sensor_link" gravity="true" collide="false" friction="0.9"/>
         <gazebo_link name="${prefix}_imu_frame" gravity="true" collide="false" friction="0.9"/>
+        <gazebo reference="base_footprint">
+          <!--
+          <kinematic>true</kinematic>
+           -->
+        </gazebo>
     </xacro:macro>
 </robot>

File: urdf/hand_v0/hand.transmission.xacro (robot description, xacro)
@@ -27,7 +27,7 @@
 <robot xmlns:xacro="http://www.ros.org/wiki.xacro">
     <xacro:macro name="hsrb_hand_transmission" params="prefix">
-        <hsrb_effort_joint_transmission joint="${prefix}_motor_joint" reduction="1"/>
-        <hsrb_effort_joint_transmission joint="${prefix}_l_spring_proximal_joint" reduction="1"/>
-        <hsrb_effort_joint_transmission joint="${prefix}_r_spring_proximal_joint" reduction="1"/>
+        <hsrb_position_joint_transmission joint="${prefix}_motor_joint" reduction="1"/>
+        <hsrb_position_joint_transmission joint="${prefix}_l_spring_proximal_joint" reduction="1"/>
+        <hsrb_position_joint_transmission joint="${prefix}_r_spring_proximal_joint" reduction="1"/>
     </xacro:macro>
 </robot>

File: urdf/sensors/rgbd_sensor.urdf.xacro (robot description, xacro)
@@ -47,16 +47,22 @@
             </collision>
         </link>
-        <joint name="${prefix}_rgbd_sensor_gazebo_frame_joint" type="fixed">
+<!--
+        <joint name="${prefix}_rgbd_sensor_frame_joint" type="fixed">
             <origin xyz="0 0 0" rpy="${pi/2.0} ${-pi/2.0} 0.0"/>
             <parent link="${prefix}_${sensor_name}_link"/>
-            <child link="${prefix}_${sensor_name}_gazebo_frame"/>
+            <child link="${prefix}_${sensor_name}_frame"/>
         </joint>
-        `
-        <link name="${prefix}_${sensor_name}_gazebo_frame"></link>
+         -->
+        <joint name="${prefix}_rgbd_sensor_frame_joint" type="fixed">
+            <origin xyz="0 0 0" rpy="0.0 0.0 0.0"/>
+            <parent link="${prefix}_${sensor_name}_link"/>
+            <child link="${prefix}_${sensor_name}_frame"/>
+        </joint>
+        <link name="${prefix}_${sensor_name}_frame"></link>
         <xacro:rgbd_sensor_gazebo
             robot_namespace="${robot_namespace}"
             sensor_name="${prefix}_${sensor_name}"
-            parent_frame="${prefix}_${sensor_name}_gazebo_frame"
-            topic_frame_id="${prefix}_${sensor_name}_rgb_frame" />
+            parent_frame="${prefix}_${sensor_name}_frame"
+            topic_frame_id="${prefix}_${sensor_name}_frame" />
     </xacro:macro>
 </robot>
